File: kicad/pq-cdh/pq-cdh.kicad_sch (KiCad schematic)
At the start: 35 parts, among them IC1 STM32L496RGT3, IC2 IS25LP128F-JBLA3, J1 Conn_01x04, J2 Conn_01x16, J3 Conn_01x04, J4 Conn_01x04, J5 Conn_01x16, J6 Conn_01x04, J7 Conn_02x06_Odd_Even, J8 Conn_01x04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

Commit message: With Changes related Ext Flash SPI configuration
Connections:
- net SPI1_NSS: now reaches IC1.26 (PB0)
- net SPI1_NSS: now also IC2.1 (CE#), R5.2
- net SPI1_SCK: now reaches IC1.55 (PB3)
- net SPI1_SCK: now also IC2.6 (SCK)
- net SPI1_MISO: now reaches IC1.56 (PB4)
- net SPI1_MISO: now also IC2.2 (SO(IO1))
- net SPI1_MOSI: now reaches IC1.57 (PB5)
- net SPI1_MOSI: now also IC2.5 (SI(IO0))
- removed net QUADSPI_BK1_NCS: IC1.16 (PA2), IC2.1 (CE#), R5.2
- net QUADSPI_BK2_IO0: no longer names the net of IC1.9 (PC1)
- net QUADSPI_BK2_IO0: no longer IC2.5 (SI(IO0))
- net QUADSPI_BK2_IO1 renamed IO1_WP
- net IO1_WP: now also IC2.3 (WP#(IO2)); no longer IC2.2 (SO(IO1))
- net QUADSPI_BK2_IO2 renamed IO2_HR
- net IO2_HR: now also IC2.7 (HOLD#_OR__RESET#(IO3)); no longer IC2.3 (WP#(IO2))
- net QUADSPI_BK2_IO3: no longer names the net of IC1.24 (PC4)
- net QUADSPI_BK2_IO3: no longer IC2.7 (HOLD#_OR__RESET#(IO3))
- net QUADSPI_CLK: no longer names the net of IC1.17 (PA3)
- net QUADSPI_CLK: no longer IC2.6 (SCK)
Changed lines of the file:
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@@
   (no_connect (at 187.96 99.06))
   (no_connect (at 187.96 101.6))
+  (no_connect (at 93.98 86.36))
   (no_connect (at 93.98 88.9))
+  (no_connect (at 93.98 68.58))
+  (no_connect (at 68.58 50.8))
   (no_connect (at 93.98 104.14))
   (no_connect (at 40.64 73.66))
   (no_connect (at 40.64 76.2))
-  (no_connect (at 68.58 129.54))
-  (no_connect (at 63.5 129.54))
-  (no_connect (at 66.04 129.54))
   (no_connect (at 50.8 129.54))
   (no_connect (at 60.96 129.54))
   (no_connect (at 58.42 50.8))
   (no_connect (at 60.96 50.8))
-  (no_connect (at 63.5 50.8))
   (no_connect (at 66.04 50.8))
   (no_connect (at 71.12 50.8))
@@
   (no_connect (at 93.98 71.12))
   (no_connect (at 93.98 73.66))
+  (no_connect (at 86.36 50.8))
   (wire (pts (xy 93.98 99.06) (xy 109.22 99.06))
     (stroke (width 0) (type default) (color 0 0 0 0))
@@
     (effects (font (size 1.27 1.27)) (justify right bottom))
   )
-  (label "QUADSPI_BK2_IO0" (at 237.49 162.56 0)
+  (label "SPI1_MOSI" (at 237.49 162.56 0)
     (effects (font (size 1.27 1.27)) (justify left bottom))
   )
@@
     (effects (font (size 1.27 1.27)) (justify left bottom))
   )
-  (label "QUADSPI_CLK" (at 86.36 50.8 90)
-    (effects (font (size 1.27 1.27)) (justify left bottom))
-  )
   (label "DCMI_D7" (at 233.68 71.12 180)
     (effects (font (size 1.27 1.27)) (justify right bottom))
   )
-  (label "QUADSPI_BK1_NCS" (at 177.8 154.94 180)
+  (label "SPI1_NSS" (at 177.8 154.94 180)
     (effects (font (size 1.27 1.27)) (justify right bottom))
   )
@@
     (effects (font (size 1.27 1.27)) (justify left bottom))
   )
-  (label "QUADSPI_BK2_IO2" (at 93.98 81.28 0)
-    (effects (font (size 1.27 1.27)) (justify left bottom))
-  )
   (label "SWCLK" (at 48.26 129.54 270)
     (effects (font (size 1.27 1.27)) (justify right bottom))
@@
     (effects (font (size 1.27 1.27)) (justify right bottom))
   )
-  (label "QUADSPI_BK2_IO0" (at 93.98 86.36 0)
-    (effects (font (size 1.27 1.27)) (justify left bottom))
-  )
   (label "DCMI_D1" (at 40.64 81.28 180)
     (effects (font (size 1.27 1.27)) (justify right bottom))
@@
     (effects (font (size 1.27 1.27)) (justify left bottom))
   )
-  (label "QUADSPI_BK2_IO3" (at 68.58 50.8 90)
-    (effects (font (size 1.27 1.27)) (justify left bottom))
-  )
   (label "DCMI_D3" (at 233.68 76.2 180)
     (effects (font (size 1.27 1.27)) (justify right bottom))
@@
   (label "DCMI_D0" (at 40.64 78.74 180)
     (effects (font (size 1.27 1.27)) (justify right bottom))
-  )
-  (label "QUADSPI_BK2_IO1" (at 93.98 83.82 0)
-    (effects (font (size 1.27 1.27)) (justify left bottom))
   )
   (label "USART1_TX" (at 40.64 91.44 180)
@@
     (effects (font (size 1.27 1.27)) (justify left bottom))
   )
-  (label "QUADSPI_BK2_IO1" (at 181.61 157.48 180)
+  (label "SPI1_MISO" (at 181.61 157.48 180)
     (effects (font (size 1.27 1.27)) (justify right bottom))
   )
@@
     (effects (font (size 1.27 1.27)) (justify right bottom))
   )
-  (label "QUADSPI_BK2_IO2" (at 181.61 160.02 180)
+  (label "SPI1_MISO" (at 66.04 129.54 270)
+    (effects (font (size 1.27 1.27)) (justify right bottom))
+  )
+  (label "IO1_WP" (at 181.61 160.02 180)
     (effects (font (size 1.27 1.27)) (justify right bottom))
   )
@@
     (effects (font (size 1.27 1.27)) (justify right bottom))
   )
+  (label "SPI1_NSS" (at 63.5 50.8 90)
+    (effects (font (size 1.27 1.27)) (justify left bottom))
+  )
   (label "LED1" (at 53.34 129.54 270)
     (effects (font (size 1.27 1.27)) (justify right bottom))
@@
     (effects (font (size 1.27 1.27)) (justify right bottom))
   )
+  (label "IO1_WP" (at 93.98 83.82 0)
+    (effects (font (size 1.27 1.27)) (justify left bottom))
+  )
   (label "LPUART_RX" (at 177.8 26.67 270)
     (effects (font (size 1.27 1.27)) (justify right bottom))
@@
   )
   (label "LED2" (at 20.32 176.53 180)
+    (effects (font (size 1.27 1.27)) (justify right bottom))
+  )
+  (label "SPI1_SCK" (at 63.5 129.54 270)
     (effects (font (size 1.27 1.27)) (justify right bottom))
   )
@@
     (effects (font (size 1.27 1.27)) (justify left bottom))
   )
-  (label "QUADSPI_CLK" (at 237.49 160.02 0)
+  (label "SPI1_SCK" (at 237.49 160.02 0)
     (effects (font (size 1.27 1.27)) (justify left bottom))
   )
@@
     (effects (font (size 1.27 1.27)) (justify right bottom))
   )
-  (label "QUADSPI_BK2_IO3" (at 237.49 157.48 0)
+  (label "IO2_HR" (at 93.98 81.28 0)
     (effects (font (size 1.27 1.27)) (justify left bottom))
   )
+  (label "IO2_HR" (at 237.49 157.48 0)
+    (effects (font (size 1.27 1.27)) (justify left bottom))
+  )
   (label "VDD_FILT" (at 95.25 182.88 180)
     (effects (font (size 1.27 1.27)) (justify right bottom))
   )
-  (label "QUADSPI_BK1_NCS" (at 93.98 68.58 0)
-    (effects (font (size 1.27 1.27)) (justify left bottom))
-  )
   (label "USART1_CK" (at 231.14 27.94 270)
+    (effects (font (size 1.27 1.27)) (justify right bottom))
+  )
+  (label "SPI1_MOSI" (at 68.58 129.54 270)
     (effects (font (size 1.27 1.27)) (justify right bottom))
   )
@@
   )
   (symbol (lib_id "pq-cdh:STM32L496RGT3") (at 93.98 106.68 180) (unit 1)
-    (in_bom yes) (on_board yes) (fields_autoplaced)
+    (in_bom yes) (on_board yes)
     (property "Reference" "IC1" (id 0) (at 97.79 62.7505 0)
       (effects (font (size 1.27 1.27)) hide)
     )
-    (property "Value" "STM32L496RGT3" (id 1) (at 97.79 65.2905 0))
+    (property "Value" "STM32L496RGT3" (id 1) (at 68.58 71.12 0))
     (property "Footprint" "pq-cdh:QFP50P1200X1200X160-64N" (id 2) (at 44.45 124.46 0)
       (effects (font (size 1.27 1.27)) (justify left) hide)
