File: kicad/pq-cdh/pq-cdh.kicad_sch (KiCad schematic)
At the start: 35 parts, among them IC1 STM32L496RGT3, IC2 IS25LP128F-JBLA3, J1 Conn_01x04, J2 Conn_01x16, J3 Conn_01x04, J4 Conn_01x04, J5 Conn_01x16, J6 Conn_01x04, J7 Conn_02x06_Odd_Even, J8 Conn_01x04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

Commit message: gerber_update
Parts:
- removed C14, C5, C6, C7, C9: 0603ZA220JAT2A, pq-cdh:CAPC1608X90N, symbol pq-cdh:0603ZA220JAT2A
- added C14, C7, C9: 0603ZC104JAT2A, CAPC1608X90N, symbol pq-cdh:0603ZC104JAT2A
- added C5, C6: 0603ZC105JAT2A, CAPC1608X90N, symbol pq-cdh:0603ZC105JAT2A
Connections:
- net GND: now also C14.2, C5.2, C6.2, C7.2, C9.2
- net NRST: now also C9.1
- net VDD_FILT: now also C14.1, C5.1, C6.1, C7.1

Commit message: pd_cdh_v0.2.0
- I2C3 SDA and SCL to pins 1 and 2 on the bottom header row
- ADC to pin 3 on the bottom header row
- unused GPIO to pins 4 and 5 on the bottom header row
Connections:
- net AIN16: now reaches IC1.27 (PB1)
- net AIN16: now also J2.3 (Pin_3)
- net IO3: now reaches IC1.50 (PA15)
- net IO3: now also J2.4 (Pin_4)
- net IO4: now reaches IC1.54 (PD2)
- net IO4: now also J2.5 (Pin_5)
- net SCL3: now reaches IC1.8 (PC0)
- net SCL3: now also J2.2 (Pin_2)
- net SDA3: now reaches IC1.9 (PC1)
- net SDA3: now also J2.1 (Pin_1)
- no-connect marks 48 -> 38
